Commit message: add ultrasonic sensor at front

File: urdf/mobile_robot.urdf.xacro (robot description, xacro)
@@ -106,3 +106,23 @@
 		</collision>
 	</link>
+	<joint name="sonar_joint" type="fixed">
+		<origin xyz="0.0 0.163 0.025" rpy="0 0 1.5708"/>
+		<parent link="base_plate_link"/>
+		<child link="sonar"/>
+	</joint>
+	<link name="sonar">
+		<visual>
+			<origin rpy="0 0 -1.5708" xyz="0.0 0.0 0.0"/>
+			<geometry>
+				<mesh filename="package://robot_driver/stl/HC-SR04.stl" scale="0.001 0.001 0.001"/>
+			</geometry>
+			<material name="white"/>
+		</visual>
+		<collision>
+			<origin rpy="0 0 1.5708" xyz="0.0 0.0 0.0"/>
+			<geometry>
+				<mesh filename="package://robot_driver/stl/HC-SR04.stl" scale="0.001 0.001 0.001"/>
+			</geometry>
+		</collision>
+	</link>
 </robot>

Commit message: add sensor addon and tf_luna range sensor node

File: urdf/mobile_robot.urdf.xacro (robot description, xacro)
@@ -106,10 +106,10 @@
 		</collision>
 	</link>
-	<joint name="sonar_joint" type="fixed">
+	<joint name="ir_joint" type="fixed">
 		<origin xyz="0.0 0.163 0.025" rpy="0 0 1.5708"/>
 		<parent link="base_plate_link"/>
-		<child link="sonar"/>
+		<child link="ir_range"/>
 	</joint>
-	<link name="sonar">
+	<link name="ir_range">
 		<visual>
 			<origin rpy="0 0 -1.5708" xyz="0.0 0.0 0.0"/>
